File: CurrentMonitor.sch (EAGLE design)
At the start: 50 parts, among them J1 Ext Pwr, U1 NCP1117DT50G, U2 MCP1700, U3 ATmega328P-PU, Y1 16MHz 18pF

Commit message: Add terminal blocks for additional GPIO and LEDs.
Parts:
- removed JP1: ICSP, _jc:AVR_SPI_PRG_62X3_LOCK
- added D11: Green, _jc:LEDD0805
- added D12: Yellow, _jc:LEDD0805
- added R13, R14: 1K, _jc:R-US_M0805
- added TB3: D2, _jc:OST-TB-23.5MM
- added TB4: D3, _jc:OST-TB-23.5MM
- added TB5: D6, _jc:OST-TB-23.5MM
- added TB6: D7, _jc:OST-TB-23.5MM
- D13: value HB -> Red
- TB1: value CT-0 -> A0
- TB2: value CT-1 -> A1
Connections:
- new net N$18: D11.A, R14.1
- new net N$9: D12.A, R13.1
- new net PD2: TB3.1, U3.PD2(INT0)
- new net PD3: TB4.1, U3.PD3(INT1)
- new net PD6: TB5.1, U3.PD6(AIN0)
- new net PD7: TB6.1, U3.PD7(AIN1)
- net /RESET: no longer JP1.RST
- net GND: now also D11.C, D12.C, TB3.2, TB4.2, TB5.2, TB6.2; no longer JP1.GND
- net MISO: now also R13.2; no longer JP1.MISO
- net MOSI: now also R14.2; no longer JP1.MOSI
- net SCK: no longer JP1.SCK
- net VCC: no longer JP1.VCC
Other:
- note added: "v1.1"
- note removed: "v1.0"

Commit message: Layout tweaks.
Parts:
- removed JP4: Run/Pgm, SparkFun:M03PTH
- added JP1: FTDI, SparkFun:M06LOCK
- C15: value 10uF -> 4.7uF
- JP2: value FTDI -> I2C; device SparkFun:M06LOCK -> SparkFun:M04LOCK
- JP3: value I2C -> Run/Pgm; device SparkFun:M04LOCK -> SparkFun:M03PTH
- R10, R9: value 2.2K -> 200
- R11, R12: value 1K -> 2.2K
- R2: value 10K -> 1K
- R4: value 1K -> 10K
- R5, R6: value 4.7K -> 1K
- R7, R8: value 200 -> 4.7K
- U2: value MCP1700 -> MCP1700T-3302E/TT
Connections:
- net +3V3: now also R7.2, R8.2; no longer R5.2, R6.2
- net /RESET: now also R4.1; no longer R2.1
- net ADC0: now also R13.2; no longer R11.2
- net ADC1: now also R14.1; no longer R12.1
- net GND: now also JP1.1, JP1.2, JP2.4, R12.1; no longer JP2.1, JP2.2, JP3.4, R10.1
- net MISO: now also R2.2; no longer R13.2
- net MOSI: now also R3.2; no longer R14.2
- net N$10: now also JP3.1; no longer JP4.1
- net N$11: now also R5.1; no longer R3.1
- net N$12: now also R6.1; no longer R4.1
- net N$13: now also R5.2; no longer R3.2
- net N$14: now also R6.2; no longer R4.2
- net N$15: now also R13.1, R9.2; no longer R11.1, R7.2
- net N$16: now also R10.1, R14.2; no longer R12.2, R8.1
- net N$17: now also R8.1; no longer R6.1
- net N$18: now also R3.1; no longer R14.1
- net N$3: now also R11.1, R12.2; no longer R7.1, R8.2
- net N$8: now also R7.1; no longer R5.1
- net N$9: now also R2.1; no longer R13.1
- net RST: now also JP1.6; no longer JP2.6
- net RXD: now also JP1.4, JP3.2; no longer JP2.4, JP4.2
- net SCL: now also JP2.1; no longer JP3.1
- net SDA: now also JP2.2; no longer JP3.2
- net TXD: now also JP1.5; no longer JP2.5
- net VCC: now also JP1.3, R11.2, R4.2; no longer JP3.3, R2.2, R9.2
Other:
- moved on the sheet: C7, D13, R1, R10, R11, R12, R13, R14, R2, R3, R4, R5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

Commit message: Change Run/Pgm header to "lock" package.
Parts:
- JP3: device SparkFun:M03PTH -> SparkFun:M03LOCK
Changed lines of the file:
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@@
 <grid distance="0.1" unitdist="inch" unit="inch" style="lines" multiple="1" display="no" altdistance="0.01" altunitdist="inch" altunit="inch"/>
 <layers>
-<layer number="1" name="Top" color="4" fill="1" visible="no" active="no"/>
-<layer number="16" name="Bottom" color="1" fill="1" visible="no" active="no"/>
-<layer number="17" name="Pads" color="2" fill="1" visible="no" active="no"/>
-<layer number="18" name="Vias" color="2" fill="1" visible="no" active="no"/>
-<layer number="19" name="Unrouted" color="6" fill="1" visible="no" active="no"/>
-<layer number="20" name="Dimension" color="15" fill="1" visible="no" active="no"/>
-<layer number="21" name="tPlace" color="7" fill="1" visible="no" active="no"/>
-<layer number="22" name="bPlace" color="7" fill="1" visible="no" active="no"/>
-<layer number="23" name="tOrigins" color="15" fill="1" visible="no" active="no"/>
-<layer number="24" name="bOrigins" color="15" fill="1" visible="no" active="no"/>
-<layer number="25" name="tNames" color="7" fill="1" visible="no" active="no"/>
-<layer number="26" name="bNames" color="7" fill="1" visible="no" active="no"/>
-<layer number="27" name="tValues" color="7" fill="1" visible="no" active="no"/>
-<layer number="28" name="bValues" color="7" fill="1" visible="no" active="no"/>
+<layer number="1" name="Top" color="4" fill="1" visible="yes" active="no"/>
+<layer number="16" name="Bottom" color="1" fill="1" visible="yes" active="no"/>
+<layer number="17" name="Pads" color="2" fill="1" visible="yes" active="no"/>
+<layer number="18" name="Vias" color="2" fill="1" visible="yes" active="no"/>
+<layer number="19" name="Unrouted" color="6" fill="1" visible="yes" active="no"/>
+<layer number="20" name="Dimension" color="15" fill="1" visible="yes" active="no"/>
+<layer number="21" name="tPlace" color="7" fill="1" visible="yes" active="no"/>
+<layer number="22" name="bPlace" color="7" fill="1" visible="yes" active="no"/>
+<layer number="23" name="tOrigins" color="15" fill="1" visible="yes" active="no"/>
+<layer number="24" name="bOrigins" color="15" fill="1" visible="yes" active="no"/>
+<layer number="25" name="tNames" color="7" fill="1" visible="yes" active="no"/>
+<layer number="26" name="bNames" color="7" fill="1" visible="yes" active="no"/>
+<layer number="27" name="tValues" color="7" fill="1" visible="yes" active="no"/>
+<layer number="28" name="bValues" color="7" fill="1" visible="yes" active="no"/>
 <layer number="29" name="tStop" color="7" fill="3" visible="no" active="no"/>
 <layer number="30" name="bStop" color="7" fill="6" visible="no" active="no"/>
@@
 <layer number="35" name="tGlue" color="7" fill="4" visible="no" active="no"/>
 <layer number="36" name="bGlue" color="7" fill="5" visible="no" active="no"/>
-<layer number="37" name="tTest" color="7" fill="1" visible="no" active="no"/>
-<layer number="38" name="bTest" color="7" fill="1" visible="no" active="no"/>
+<layer number="37" name="tTest" color="7" fill="1" visible="yes" active="no"/>
+<layer number="38" name="bTest" color="7" fill="1" visible="yes" active="no"/>
 <layer number="39" name="tKeepout" color="4" fill="11" visible="no" active="no"/>
 <layer number="40" name="bKeepout" color="1" fill="11" visible="no" active="no"/>
@@
 <layer number="44" name="Drills" color="7" fill="1" visible="no" active="no"/>
 <layer number="45" name="Holes" color="7" fill="1" visible="no" active="no"/>
-<layer number="46" name="Milling" color="3" fill="1" visible="no" active="no"/>
-<layer number="47" name="Measures" color="7" fill="1" visible="no" active="no"/>
-<layer number="48" name="Document" color="7" fill="1" visible="no" active="no"/>
-<layer number="49" name="Reference" color="7" fill="1" visible="no" active="no"/>
-<layer number="50" name="dxf" color="7" fill="1" visible="no" active="no"/>
-<layer number="51" name="tDocu" color="7" fill="1" visible="no" active="no"/>
-<layer number="52" name="bDocu" color="7" fill="1" visible="no" active="no"/>
-<layer number="53" name="tGND_GNDA" color="7" fill="9" visible="no" active="no"/>
-<layer number="54" name="bGND_GNDA" color="1" fill="9" visible="no" active="no"/>
-<layer number="56" name="wert" color="7" fill="1" visible="no" active="no"/>
+<layer number="46" name="Milling" color="3" fill="1" visible="yes" active="no"/>
+<layer number="47" name="Measures" color="7" fill="1" visible="yes" active="no"/>
+<layer number="48" name="Document" color="7" fill="1" visible="yes" active="no"/>
+<layer number="49" name="Reference" color="7" fill="1" visible="yes" active="no"/>
+<layer number="50" name="dxf" color="7" fill="1" visible="yes" active="no"/>
+<layer number="51" name="tDocu" color="7" fill="1" visible="yes" active="no"/>
+<layer number="52" name="bDocu" color="7" fill="1" visible="yes" active="no"/>
+<layer number="53" name="tGND_GNDA" color="7" fill="9" visible="yes" active="no"/>
+<layer number="54" name="bGND_GNDA" color="1" fill="9" visible="yes" active="no"/>
+<layer number="56" name="wert" color="7" fill="1" visible="yes" active="no"/>
 <layer number="90" name="Modules" color="5" fill="1" visible="yes" active="yes"/>
 <layer number="91" name="Nets" color="2" fill="1" visible="yes" active="yes"/>
@@
 <part name="GND11" library="supply1" deviceset="GND" device=""/>
 <part name="GND12" library="supply1" deviceset="GND" device=""/>
-<part name="JP3" library="SparkFun" deviceset="M03" device="PTH" value="Run/Pgm"/>
+<part name="JP3" library="SparkFun" deviceset="M03" device="LOCK" value="Run/Pgm"/>
 <part name="D4" library="_jc" deviceset="DIODE" device="SOD-323F-A" value="1N4148"/>
 <part name="R7" library="_jc" deviceset="R-US_" device="M0805" value="4.7K"/>
